Commit message: inertia frames fixed and commands tweaked

File: resources/robots/go_bdx/go_bdx.urdf (robot description, URDF)
Before this commit: robot bdx, 19 links, 18 joints
Links:
- link head: mass 1e-9 -> None
- link head_body_pitch: mass 0.5232206536385304 -> 0.200
- link head_body_roll: mass 5.0942155694527305 -> 0.4
- link head_body_yaw: mass 0.7884788831732902 -> 0.200
- link left_foot: mass 1e-9 -> None
- link left_foot_link: mass 2.196651599731846 -> 0.678
- link left_hip: mass 1.2525665319575872 -> 0.633
- link left_hip_rotation: mass 2.7104129345182724 -> 0.633
- link left_shin: mass 3.533655907847469 -> 0.633
- link left_thigh: mass 9.79771075244762 -> 0.633
- link neck: mass 1.8541562983293536 -> 0.633
- link pelvis: mass 58.84451460019125 -> 5.713
- link right_foot: mass 1e-9 -> None
- link right_foot_link: mass 2.196651599731845 -> 0.678
- link right_hip: mass 1.2525665319575874 -> 0.633
- link right_hip_rotation: mass 2.710413234826848 -> 0.633
- link right_shin: mass 3.5336559525083544 -> 0.633
- link right_thigh: mass 9.797710752447612 -> 0.633
- link trunk: mass 1e-9 -> None

Commit message: Updated to use Duck v4

File: resources/robots/go_bdx/go_bdx.urdf (robot description, URDF)
Before this commit: robot bdx, 19 links, 18 joints
Links:
- added link ear_left, mass 0.09640158820730847; collision mesh filename=meshes/ear_left.stl scale=0.001 0.001 0.001; visual mesh filename=meshes/ear_left.stl scale=0.001 0.001 0.001
- added link ear_right, mass 0.09640158820730861; collision mesh filename=meshes/ear_right.stl scale=0.001 0.001 0.001; visual mesh filename=meshes/ear_right.stl scale=0.001 0.001 0.001
- link head: mass None -> 1e-9
- link head_body_pitch: geometry collision mesh filename=meshes/head_body_pitch.stl scale=0.001 0.001 0.001; visual mesh filename=meshes/head_body_pitch.stl scale=0.001 0.001 0.001
- link head_body_roll: geometry collision mesh filename=meshes/head_body_roll.stl scale=0.001 0.001 0.001; visual mesh filename=meshes/head_body_roll.stl scale=0.001 0.001 0.001
- link head_body_yaw: geometry collision mesh filename=meshes/head_body_yaw.stl scale=0.001 0.001 0.001; visual mesh filename=meshes/head_body_yaw.stl scale=0.001 0.001 0.001
- link left_foot: mass None -> 1e-9
- link left_foot_link: geometry collision mesh filename=meshes/left_foot.stl scale=0.001 0.001 0.001; visual mesh filename=meshes/left_foot.stl scale=0.001 0.001 0.001
- link left_hip: geometry collision mesh filename=meshes/left_hip.stl scale=0.001 0.001 0.001; visual mesh filename=meshes/left_hip.stl scale=0.001 0.001 0.001
- link left_hip_rotation: geometry collision mesh filename=meshes/left_hip_rotation.stl scale=0.001 0.001 0.001; visual mesh filename=meshes/left_hip_rotation.stl scale=0.001 0.001 0.001
- link left_shin: geometry collision mesh filename=meshes/left_shin.stl scale=0.001 0.001 0.001; visual mesh filename=meshes/left_shin.stl scale=0.001 0.001 0.001
- link left_thigh: geometry collision mesh filename=meshes/left_thigh.stl scale=0.001 0.001 0.001; visual mesh filename=meshes/left_thigh.stl scale=0.001 0.001 0.001
- link neck: geometry collision mesh filename=meshes/neck.stl scale=0.001 0.001 0.001; visual mesh filename=meshes/neck.stl scale=0.001 0.001 0.001
- link pelvis: geometry collision mesh filename=meshes/pelvis.stl scale=0.001 0.001 0.001; visual mesh filename=meshes/pelvis.stl scale=0.001 0.001 0.001
- link right_foot: mass None -> 1e-9
- link right_foot_link: geometry collision mesh filename=meshes/right_foot.stl scale=0.001 0.001 0.001; visual mesh filename=meshes/right_foot.stl scale=0.001 0.001 0.001
- link right_hip: geometry collision mesh filename=meshes/right_hip.stl scale=0.001 0.001 0.001; visual mesh filename=meshes/right_hip.stl scale=0.001 0.001 0.001
- link right_hip_rotation: geometry collision mesh filename=meshes/right_hip_rotation.stl scale=0.001 0.001 0.001; visual mesh filename=meshes/right_hip_rotation.stl scale=0.001 0.001 0.001
- link right_shin: geometry collision mesh filename=meshes/right_shin.stl scale=0.001 0.001 0.001; visual mesh filename=meshes/right_shin.stl scale=0.001 0.001 0.001
- link right_thigh: geometry collision mesh filename=meshes/right_thigh.stl scale=0.001 0.001 0.001; visual mesh filename=meshes/right_thigh.stl scale=0.001 0.001 0.001
- link trunk: mass None -> 1e-9
Joints:
- added joint left_antenna: type revolute, parent head_body_roll, child ear_left, origin xyz=-0.16665 0.0683 0.001231 rpy=0 0 0, axis -0.0 -1.0 -0.0, limit lower=-0.7853982 upper=0.7853982 effort=15 velocity=20
- added joint right_antenna: type revolute, parent head_body_roll, child ear_right, origin xyz=-0.16665 -0.0697 0.001231 rpy=0 0 0, axis -0.0 -1.0 -0.0, limit lower=-0.7853982 upper=0.7853982 effort=15 velocity=20
- joint head_frame: origin xyz=-0.03 0 0.05 rpy=0 0 -3.1415927 -> xyz=-0.03 0 0.05 rpy=0 0 0
- joint head_pitch: axis 1. 0. 0. -> -0.0 -1.0 0.0; origin xyz=-0.0013 0.064983 -0.110687 rpy=3.1415927 0.0000001 3.1415927 -> xyz=-0.065022 -0.01175 0.11088 rpy=0 0 0
- joint head_roll: axis 1. 0. 0. -> 1.0 -0.0 0.0; origin xyz=0.02964 0.045548 0.00005  rpy=1.5706214 -0. 1.5706214 -> xyz=0.039892 0.0 0.02715 rpy=0 0 0
- joint head_yaw: axis 1. 0. 0. -> -0.0 -0.0 1.0; origin xyz=0. -0.000299 0.0271  rpy=0. -1.5707963 0.  -> xyz=0.000299 0.0007 0.02897 rpy=0 0 0
- joint left_ankle: axis 1. 0. 0. -> 0.0 1.0 -0.0; origin xyz=0.011991 -0.045007 0.130142 rpy=3.1415927 0.0000001 3.1415927 -> xyz=0.045 -0.0152 -0.13 rpy=0 0 0
- joint left_foot_frame: origin xyz=-0.015 -0.02 -0.08027 rpy=0 0 -1.57079632679489 -> xyz=0.0 0.0 -0.075 rpy=0 0 0
- joint left_hip_pitch: axis 1. 0. 0. -> 0.0 1.0 0.0; origin xyz=0.004977 0.079601 0.000749 rpy=0. 0. 1.5707964 -> xyz=0.017466 0.069601 0.000785 rpy=0 0 0
- joint left_hip_roll: axis 1. 0. 0. -> 1.0 -0.0 -0.0; origin xyz=0.06335 -0.0052 0.00275 rpy=1.5707964 0. -1.5707964 -> xyz=-0.0073 0.00275 -0.076 rpy=0 0 0
- joint left_hip_yaw: axis 1. 0. 0. -> -0.0 0.0 -1.0; limit lower=-0.2617994 upper=0.2617994 effort=23.7 velocity=30 -> lower=-0.7853982 upper=0.7853982 effort=23.7 velocity=30; origin xyz=0.046658 0.013027 0.350727 rpy=0. 1.5707963 0.  -> xyz=-0.033111 0.046658 0.363959 rpy=0 0 0
- joint left_knee: axis 1. 0. 0. -> -0.0 -1.0 0.0; origin xyz=0. 0.079306 -0.077708 rpy=3.1415927 -0.0000001 3.1415927 -> xyz=-0.079306 0.0 -0.077708 rpy=0 0 0
- joint neck_pitch: axis 1. 0. 0. -> -0.0 -1.0 0.0; origin xyz=-0.0013 -0.076423 0.394589 rpy=3.1415927 -0.0000001 3.1415927 -> xyz=0.056339 0.0119 0.395171 rpy=0 0 0
- joint right_ankle: axis 1. 0. 0. -> -0.0 -1.0 0.0; origin xyz=0.011991 -0.045007 -0.130142 rpy=3.1415927 -0.0000001 3.1415927 -> xyz=0.045 0.0152 -0.13 rpy=0 0 0
- joint right_foot_frame: origin xyz=-0.015 -0.02 0.0802759 rpy=3.141592653589 0 -1.570796326794 -> xyz=0.0 0.0 -0.075 rpy=0 0 0
- joint right_hip_pitch: axis 1. 0. 0. -> -0.0 -1.0 0.0; origin xyz=0.004977 -0.079601 0.000749 rpy=3.1415927 -0.0000001 -1.5707964 -> xyz=0.017466 -0.069601 0.000785 rpy=0 0 0
- joint right_hip_roll: axis 1. 0. 0. -> 1.0 -0.0 -0.0; origin xyz=0.06335 -0.0052 -0.00275 rpy=1.5707964 0. -1.5707964 -> xyz=-0.0073 -0.00275 -0.076 rpy=0 0 0
- joint right_hip_yaw: axis 1. 0. 0. -> -0.0 -0.0 -1.0; limit lower=-0.2617994 upper=0.2617994 effort=23.7 velocity=30 -> lower=-0.7853982 upper=0.7853982 effort=23.7 velocity=30; origin xyz=-0.046658 0.013027 0.350727 rpy=0. 1.5707963 0.  -> xyz=-0.033111 -0.046658 0.363959 rpy=0 0 0
- joint right_knee: axis 1. 0. 0. -> 0.0 1.0 -0.0; origin xyz=-0. 0.079306 0.077708 rpy=3.1415927 0.0000001 3.1415927 -> xyz=-0.079306 0.0 -0.077708 rpy=0 0 0
- joint trunk_frame: origin xyz=0 0 0.35 rpy=0 0 -1.5707963267948 -> xyz=-0.035 0 0.29 rpy=0 0 0

Commit message: Updated walk data and offsets

File: resources/robots/go_bdx/go_bdx.urdf (robot description, URDF)
Before this commit: robot bdx, 21 links, 20 joints
Joints:
- joint trunk_frame: origin xyz=-0.035 0 0.29 rpy=0 0 0 -> xyz=-0.035 0 0.2695 rpy=0 0 0

Commit message: Updated parameters

File: resources/robots/go_bdx/go_bdx.urdf (robot description, URDF)
Before this commit: robot bdx, 21 links, 20 joints
Joints:
- joint trunk_frame: origin xyz=-0.035 0 0.2695 rpy=0 0 0 -> xyz=-0.035 0 0.26943 rpy=0 0 0

Commit message: Updating parameters

File: resources/robots/go_bdx/go_bdx.urdf (robot description, URDF)
Before this commit: robot bdx, 21 links, 20 joints
Joints:
- joint head_pitch: limit lower=-0.7853982 upper=0.7853982 effort=15 velocity=20 -> lower=-0.7853982 upper=0.7853982 effort=7.3 velocity=5.55
- joint head_roll: limit lower=-0.7853982 upper=0.7853982 effort=15 velocity=20 -> lower=-0.7853982 upper=0.7853982 effort=7.3 velocity=5.55
- joint head_yaw: limit lower=-0.7853982 upper=0.7853982 effort=15 velocity=20 -> lower=-0.7853982 upper=0.7853982 effort=7.3 velocity=5.55
- joint left_antenna: limit lower=-0.7853982 upper=0.7853982 effort=15 velocity=20 -> lower=-0.7853982 upper=0.7853982 effort=0.2943 velocity=13.62
- joint left_foot_frame: origin xyz=0.0 0.0 -0.075 rpy=0 0 0 -> xyz=0.025 0.0 -0.0765 rpy=0 0 0
- joint right_antenna: limit lower=-0.7853982 upper=0.7853982 effort=15 velocity=20 -> lower=-0.7853982 upper=0.7853982 effort=0.2943 velocity=13.62
- joint right_foot_frame: origin xyz=0.0 0.0 -0.075 rpy=0 0 0 -> xyz=0.025 0.0 -0.0765 rpy=0 0 0

Commit message: Updated parameters

File: resources/robots/go_bdx/go_bdx.urdf (robot description, URDF)
Before this commit: robot bdx, 21 links, 20 joints
Joints:
- joint left_foot_frame: origin xyz=0.025 0.0 -0.0765 rpy=0 0 0 -> xyz=0.025 0.0 -0.0785 rpy=0 0 0
- joint right_foot_frame: origin xyz=0.025 0.0 -0.0765 rpy=0 0 0 -> xyz=0.025 0.0 -0.0785 rpy=0 0 0
