Commit message: correct torque and velocities in urdf

File: resources/robots/bdx/urdf/bdx.urdf (robot description, URDF)
Before this commit: robot bdx, 20 links, 19 joints
Joints:
- joint left_ankle: limit lower=-1.570796326794896558 upper=1.570796326794896558 effort=0.52 velocity=10.7 -> lower=-1.570796326794896558 upper=1.570796326794896558 effort=0.93 velocity=8.48
- joint left_antenna: limit lower=-1.1344640137963142301 upper=2.0943951023931952626 effort=0.52 velocity=10.7 -> lower=-1.1344640137963142301 upper=2.0943951023931952626 effort=0.17 velocity=10
- joint left_hip_pitch: limit lower=-0.52359877559829881566 upper=1.570796326794896558 effort=0.52 velocity=10.7 -> lower=-0.52359877559829881566 upper=1.570796326794896558 effort=0.93 velocity=8.48
- joint left_hip_roll: limit lower=-1.570796326794896558 upper=0.43633231299858238339 effort=0.52 velocity=10.7 -> lower=-1.570796326794896558 upper=0.43633231299858238339 effort=0.93 velocity=8.48
- joint left_hip_yaw: limit lower=-0.69813170079773179122 upper=0.69813170079773179122 effort=0.52 velocity=10.7 -> lower=-0.69813170079773179122 upper=0.69813170079773179122 effort=0.93 velocity=8.48
- joint left_knee: limit lower=-2.0943951023931952626 upper=2.0943951023931952626 effort=0.52 velocity=10.7 -> lower=-2.0943951023931952626 upper=2.0943951023931952626 effort=0.93 velocity=8.48
- joint right_ankle: limit lower=-1.570796326794896558 upper=1.570796326794896558 effort=0.52 velocity=10.7 -> lower=-1.570796326794896558 upper=1.570796326794896558 effort=0.93 velocity=8.48
- joint right_antenna: limit lower=-2.0943951023931952626 upper=1.1344640137963142301 effort=0.52 velocity=10.7 -> lower=-2.0943951023931952626 upper=1.1344640137963142301 effort=0.17 velocity=10
- joint right_hip_pitch: limit lower=-0.52359877559829881566 upper=1.570796326794896558 effort=0.52 velocity=10.7 -> lower=-0.52359877559829881566 upper=1.570796326794896558 effort=0.93 velocity=8.48
- joint right_hip_roll: limit lower=-1.570796326794896558 upper=0.43633231299858238339 effort=0.52 velocity=10.7 -> lower=-1.570796326794896558 upper=0.43633231299858238339 effort=0.93 velocity=8.48
- joint right_hip_yaw: limit lower=-0.69813170079773179122 upper=0.69813170079773179122 effort=0.52 velocity=10.7 -> lower=-0.69813170079773179122 upper=0.69813170079773179122 effort=0.93 velocity=8.48
- joint right_knee: limit lower=-2.0943951023931952626 upper=2.0943951023931952626 effort=0.52 velocity=10.7 -> lower=-2.0943951023931952626 upper=2.0943951023931952626 effort=0.93 velocity=8.48

Commit message: Updated

File: resources/robots/bdx/urdf/bdx.urdf (robot description, URDF)
Before this commit: robot bdx, 20 links, 19 joints
Joints:
- joint left_ankle: limit lower=-1.570796326794896558 upper=1.570796326794896558 effort=0.52 velocity=10.7 -> lower=-1.570796326794896558 upper=1.570796326794896558 effort=0.93 velocity=8.48
- joint left_hip_pitch: limit lower=-0.52359877559829881566 upper=1.570796326794896558 effort=0.52 velocity=10.7 -> lower=-0.52359877559829881566 upper=1.570796326794896558 effort=0.93 velocity=8.48
- joint left_hip_roll: limit lower=-1.570796326794896558 upper=0.43633231299858238339 effort=0.52 velocity=10.7 -> lower=-1.570796326794896558 upper=0.43633231299858238339 effort=0.93 velocity=8.48
- joint left_hip_yaw: limit lower=-0.69813170079773179122 upper=0.69813170079773179122 effort=0.52 velocity=10.7 -> lower=-0.69813170079773179122 upper=0.69813170079773179122 effort=0.93 velocity=8.48
- joint left_knee: limit lower=-2.0943951023931952626 upper=2.0943951023931952626 effort=0.52 velocity=10.7 -> lower=-2.0943951023931952626 upper=2.0943951023931952626 effort=0.93 velocity=8.48
- joint right_ankle: limit lower=-1.570796326794896558 upper=1.570796326794896558 effort=0.52 velocity=10.7 -> lower=-1.570796326794896558 upper=1.570796326794896558 effort=0.93 velocity=8.48
- joint right_hip_pitch: limit lower=-0.52359877559829881566 upper=1.570796326794896558 effort=0.52 velocity=10.7 -> lower=-0.52359877559829881566 upper=1.570796326794896558 effort=0.93 velocity=8.48
- joint right_hip_roll: limit lower=-1.570796326794896558 upper=0.43633231299858238339 effort=0.52 velocity=10.7 -> lower=-1.570796326794896558 upper=0.43633231299858238339 effort=0.93 velocity=8.48
- joint right_hip_yaw: limit lower=-0.69813170079773179122 upper=0.69813170079773179122 effort=0.52 velocity=10.7 -> lower=-0.69813170079773179122 upper=0.69813170079773179122 effort=0.93 velocity=8.48
- joint right_knee: limit lower=-2.0943951023931952626 upper=2.0943951023931952626 effort=0.52 velocity=10.7 -> lower=-2.0943951023931952626 upper=2.0943951023931952626 effort=0.93 velocity=8.48
